Commit message: Fix: apriltag localization tf fix

File: pangolin_description/urdf/pangolin_urdf_20240701.urdf (robot description, URDF)
Before this commit: robot pangolin_urdf_20240701, 10 links, 9 joints
Joints:
- joint cam_joint: origin xyz=0.0257215676729172 -4.25630967756469E-05 0.0528721377651949 rpy=1.5707963267949 3.141592654 1.5707963267949 -> xyz=0.0257215676729172 -4.25630967756469E-05 0.0528721377651949 rpy=3.141592654 3.141592654 3.141592654

Commit message: Feat: AprilTag localization

File: pangolin_description/urdf/pangolin_urdf_20240701.urdf (robot description, URDF)
Before this commit: robot pangolin_urdf_20240701, 10 links, 9 joints
Links:
- removed link backbody_Link
- removed link head_Link
- removed link lf_Link
- removed link middle_Link
- removed link rb_Link
- removed link rf_Link
- added link backbody_link, mass 0.133315232250175; collision mesh filename=package://pangolin_description/meshes/backbody_Link.STL; visual mesh filename=package://pangolin_description/meshes/backbody_Link.STL
- added link head_link, mass 0.0552741565417432; collision mesh filename=package://pangolin_description/meshes/head_Link.STL; visual mesh filename=package://pangolin_description/meshes/head_Link.STL
- added link lf_link, mass 0.0475547576628768; collision mesh filename=package://pangolin_description/meshes/lf_Link.STL; visual mesh filename=package://pangolin_description/meshes/lf_Link.STL
- added link middle_link, mass 0.0516800335523288; collision mesh filename=package://pangolin_description/meshes/middle_Link.STL; visual mesh filename=package://pangolin_description/meshes/middle_Link.STL
- added link rb_link, mass 0.0475552016041672; collision mesh filename=package://pangolin_description/meshes/rb_Link.STL; visual mesh filename=package://pangolin_description/meshes/rb_Link.STL
- added link rf_link, mass 0.0475588832380788; collision mesh filename=package://pangolin_description/meshes/rf_Link.STL; visual mesh filename=package://pangolin_description/meshes/rf_Link.STL
Joints:
- removed joint rb_link
- added joint rb_joint: type continuous, parent backbody_link, child rb_link, origin xyz=-0.055701668245708 0.00208974071688019 0.0523614811329654 rpy=0 0 0, axis 0 0 1
- joint backbody_joint: child backbody_Link -> backbody_link; parent middle_Link -> middle_link
- joint head_joint: child head_Link -> head_link
- joint middle_joint: child middle_Link -> middle_link
- joint rf_joint: child rf_Link -> rf_link

Commit message: Feat: Bind_usb_rule

File: pangolin_description/urdf/pangolin_urdf_20240701.urdf (robot description, URDF)
Before this commit: robot pangolin_urdf_20240701, 10 links, 9 joints
Links:
- removed link backbody_link
- removed link head_link
- removed link lf_link
- removed link middle_link
- removed link rb_link
- removed link rf_link
- added link backbody_Link, mass 0.133315232250175; collision mesh filename=package://pangolin_description/meshes/backbody_Link.STL; visual mesh filename=package://pangolin_description/meshes/backbody_Link.STL
- added link head_Link, mass 0.0552741565417432; collision mesh filename=package://pangolin_description/meshes/head_Link.STL; visual mesh filename=package://pangolin_description/meshes/head_Link.STL
- added link lf_Link, mass 0.0475547576628768; collision mesh filename=package://pangolin_description/meshes/lf_Link.STL; visual mesh filename=package://pangolin_description/meshes/lf_Link.STL
- added link middle_Link, mass 0.0516800335523288; collision mesh filename=package://pangolin_description/meshes/middle_Link.STL; visual mesh filename=package://pangolin_description/meshes/middle_Link.STL
- added link rb_Link, mass 0.0475552016041672; collision mesh filename=package://pangolin_description/meshes/rb_Link.STL; visual mesh filename=package://pangolin_description/meshes/rb_Link.STL
- added link rf_Link, mass 0.0475588832380788; collision mesh filename=package://pangolin_description/meshes/rf_Link.STL; visual mesh filename=package://pangolin_description/meshes/rf_Link.STL
Joints:
- removed joint rb_joint
- added joint rb_link: type continuous, parent backbody_Link, child rb_Link, origin xyz=-0.055701668245708 0.00208974071688019 0.0523614811329654 rpy=0 0 0, axis 0 0 1
- joint backbody_joint: child backbody_link -> backbody_Link; parent middle_link -> middle_Link
- joint head_joint: child head_link -> head_Link
- joint middle_joint: child middle_link -> middle_Link
- joint rf_joint: child rf_link -> rf_Link

Commit message: faet: turn on vslam imu mode & add imu_link in urdf

File: pangolin_description/urdf/pangolin_urdf_20240701.urdf (robot description, URDF)
Before this commit: robot pangolin_urdf_20240701, 10 links, 9 joints
Links:
- added link imu_link, mass 0.001; collision box size=0.01 0.01 0.01; visual box size=0.01 0.01 0.01
Joints:
- added joint imu_joint: type fixed, parent base_link, child imu_link, origin xyz=0 0 0 rpy=0 0 0
